Commit message: remplacement ddbot par ddzz

File: ddbot_description/urdf/robot.urdf (robot description, URDF)
Before this commit: robot ddbot, 3 links, 2 joints
Links:
- link base_link: geometry collision mesh filename=package://ddzz_description/meshes/body.stl scale=0.001 0.001 0.001; visual mesh filename=package://ddzz_description/meshes/body.stl scale=0.001 0.001 0.001
- link left_wheel: geometry collision cylinder length=0.016 radius=0.0254; visual mesh filename=package://ddzz_description/meshes/wheel.stl scale=0.001 0.001 0.001
- link right_wheel: geometry collision cylinder length=0.016 radius=0.0254; visual mesh filename=package://ddzz_description/meshes/wheel.stl scale=0.001 0.001 0.001
